Commit message: added IMU links and joints

File: orbbec_description/urdf/gemini_335_336.urdf.xacro (robot description, xacro)
@@ -304,3 +304,31 @@
         <axis xyz="0 0 0" />
     </joint>
+    <link name="camera_accel_frame" />
+    <link name="camera_accel_optical_frame" />
+    <link name="camera_gyro_frame" />
+    <link name="camera_gyro_optical_frame" />
+    <joint name="camera_accel_joint" type="fixed">
+        <origin xyz="0 0 0" rpy="0 0 0" />
+        <parent link="camera_link" />
+        <child link="camera_accel_frame" />
+        <axis xyz="0 0 0" />
+    </joint>
+    <joint name="camera_accel_optical_joint" type="fixed">
+        <origin xyz="0 0 0" rpy="-1.5707963267949 0 -1.5707963267949" />
+        <parent link="camera_accel_frame" />
+        <child link="camera_accel_optical_frame" />
+        <axis xyz="0 0 0" />
+    </joint>
+    <joint name="camera_gyro_joint" type="fixed">
+        <origin xyz="0 0 0" rpy="0 0 0" />
+        <parent link="camera_link" />
+        <child link="camera_gyro_frame" />
+        <axis xyz="0 0 0" />
+    </joint>
+    <joint name="camera_gyro_optical_joint" type="fixed">
+        <origin xyz="0 0 0" rpy="-1.5707963267949 0 -1.5707963267949" />
+        <parent link="camera_gyro_frame" />
+        <child link="camera_gyro_optical_frame" />
+        <axis xyz="0 0 0" />
+    </joint>
 </robot>

File: orbbec_description/urdf/gemini_335_L_336_L.urdf.xacro (robot description, xacro)
@@ -522,3 +522,63 @@
       xyz="0 0 0" />
   </joint>
+  <link
+    name="camera_accel_frame" />
+  <joint
+    name="camera_accel_joint"
+    type="fixed">
+    <origin
+      xyz="0 0 0"
+      rpy="0 0 0" />
+    <parent
+      link="camera_IMU_frame" />
+    <child
+      link="camera_accel_frame" />
+    <axis
+      xyz="0 0 0" />
+  </joint>
+  <link
+    name="camera_accel_optical_frame" />
+  <joint
+    name="camera_accel_optical_joint"
+    type="fixed">
+    <origin
+      xyz="0 0 0"
+      rpy="-1.5708 0 -1.5708" />
+    <parent
+      link="camera_accel_frame" />
+    <child
+      link="camera_accel_optical_frame" />
+    <axis
+      xyz="0 0 0" />
+  </joint>
+  <link
+    name="camera_gyro_frame" />
+  <joint
+    name="camera_gyro_joint"
+    type="fixed">
+    <origin
+      xyz="0 0 0"
+      rpy="0 0 0" />
+    <parent
+      link="camera_IMU_frame" />
+    <child
+      link="camera_gyro_frame" />
+    <axis
+      xyz="0 0 0" />
+  </joint>
+  <link
+    name="camera_gyro_optical_frame" />
+  <joint
+    name="camera_gyro_optical_joint"
+    type="fixed">
+    <origin
+      xyz="0 0 0"
+      rpy="-1.5708 0 -1.5708" />
+    <parent
+      link="camera_gyro_frame" />
+    <child
+      link="camera_gyro_optical_frame" />
+    <axis
+      xyz="0 0 0" />
+  </joint>
 </robot>
