Commit message: Fixed major issue with the location of root link and added missin depth_optical link for Gemini 335L and 336L cameras.   Most of the other models have same issue with the root link but those are not fixed yet.

File: orbbec_description/urdf/gemini_335_L_336_L.urdf.xacro (robot description, xacro)
@@ -46,5 +46,5 @@
   </link>
   <link
-    name="camera_color_screw_frame">
+    name="camera_bottom_screw_frame">
     <inertial>
       <origin
@@ -86,13 +86,13 @@
   </link>
   <joint
-    name="camera_color_screw_joint"
-    type="fixed">
-    <origin
-      xyz="-0.011715 -0.0475 -0.014311"
+    name="camera_bottom_screw_joint"
+    type="fixed">
+    <origin
+      xyz="0.011715 0.0475 0.014311"
       rpy="0 0 0" />
     <parent
+      link="camera_bottom_screw_frame" />
+    <child
       link="camera_link" />
-    <child
-      link="camera_color_screw_frame" />
     <axis
       xyz="0 0 0" />
@@ -145,5 +145,5 @@
       rpy="0 0 0" />
     <parent
-      link="camera_depth_frame" />
+      link="camera_link" />
     <child
       link="camera_IMU_frame" />
@@ -205,4 +205,57 @@
   </joint>
   <link
+    name="camera_depth_optical_frame">
+    <inertial>
+      <origin
+        xyz="-0.00158020638644197 -1.72113892998871E-08 -1.52265896501485E-07"
+        rpy="0 0 0" />
+      <mass
+        value="0.00045316775745635" />
+      <inertia
+        ixx="4.34107394943177E-09"
+        ixy="-3.70457372455813E-13"
+        ixz="-1.46474854133768E-13"
+        iyy="4.84011101176503E-09"
+        iyz="2.21976196909378E-14"
+        izz="4.84043649602512E-09" />
+    </inertial>
+    <visual>
+      <origin
+        xyz="0 0 0"
+        rpy="0 0 0" />
+      <geometry>
+        <mesh
+          filename="${mesh_path}camera_depth_frame.STL" />
+      </geometry>
+      <material
+        name="">
+        <color
+          rgba="0.792156862745098 0.819607843137255 0.933333333333333 1" />
+      </material>
+    </visual>
+    <collision>
+      <origin
+        xyz="0 0 0"
+        rpy="0 0 0" />
+      <geometry>
+        <mesh
+          filename="${mesh_path}camera_depth_frame.STL" />
+      </geometry>
+    </collision>
+  </link>
+  <joint
+    name="camera_depth_optical_joint"
+    type="fixed">
+    <origin
+      xyz="0 0 0"
+      rpy="-1.5708 0 -1.5708" />
+    <parent
+      link="camera_depth_frame" />
+    <child
+      link="camera_depth_optical_frame" />
+    <axis
+      xyz="0 0 0" />
+  </joint>
+  <link
     name="camera_left_ir_frame">
     <inertial>
@@ -463,5 +516,5 @@
       rpy="0.0010157 0 0" />
     <parent
-      link="camera_depth_frame" />
+      link="camera_link" />
     <child
       link="camera_color_frame" />
